Commit message: preparing gazebo sim

File: src/lv1/robot_description/urdf/bob_ros_gz_urdf.xacro (robot description, xacro)
@@ -1,120 +1,96 @@
 <?xml version="1.0"?>
 <robot xmlns:xacro="http://www.ros.org/wiki/xacro">
-    <gazebo reference="base_link">
-        <material>Gazebo/Red</material>
-    </gazebo>
-    <gazebo reference="front_left_wheel">
-        <material>Gazebo/Black</material>
-    </gazebo>
-    <gazebo reference="front_right_wheel">
-        <material>Gazebo/Black</material>
-    </gazebo>
-    <gazebo reference="back_left_wheel">
-        <material>Gazebo/Black</material>
-    </gazebo>
-    <gazebo reference="back_right_wheel">
-        <material>Gazebo/Black</material>
-    </gazebo>
-    <gazebo reference="lidar_link">
-        <material>Gazebo/Black</material>
-    </gazebo>
-    <gazebo reference="camera_link">
-        <material>Gazebo/Black</material>
-    </gazebo>
-    <gazebo>
-        <plugin name="skid_steer_drive_controller" filename="libgazebo_ros_skid_steer_drive.so">
-            <updateRate>100.0</updateRate>
-            <robotNamespace>/</robotNamespace>
-            <leftFrontJoint>front_left_wheel_joint</leftFrontJoint>
-            <rightFrontJoint>front_right_wheel_joint</rightFrontJoint>
-            <leftRearJoint>back_left_wheel_joint</leftRearJoint>
-            <rightRearJoint>back_right_wheel_joint</rightRearJoint>
-            <wheelSeparation>0.3</wheelSeparation>
-            <wheelDiameter>0.2</wheelDiameter>
-            <robotBaseFrame>base_link</robotBaseFrame>
-            <torque>20</torque>
-            <commandTopic >cmd_vel</commandTopic >
-            <odometryTopic>odom</odometryTopic>
-            <odometryFrame>odom</odometryFrame>
-            <broadcastTF>true</broadcastTF>
-            <!-- Set to true to publish transforms for the wheel links, defaults to false -->
-            <publishWheelTF>true</publishWheelTF>
-            <!-- Set to true to publish transforms for the odometry, defaults to true -->
-            <publishOdom>true</publishOdom>
-            <!-- Set to true to publish sensor_msgs/JointState on /joint_states for the wheel joints, defaults to false -->
-            <publishWheelJointState>true</publishWheelJointState>
-        </plugin>
-    </gazebo>
-    <gazebo reference="lidar_link">
-        <sensor type="ray" name="head_hokuyo_sensor">
-        <pose>0 0 0 0 0 0</pose>
-        <visualize>false</visualize>
-        <update_rate>40</update_rate>
-        <ray>
-            <scan>
-                <horizontal>
-                    <samples>720</samples>
-                    <resolution>1</resolution>
-                    <min_angle>-3.14</min_angle>
-                    <max_angle>3.14</max_angle>
-                </horizontal>
-            </scan>
-            <range>
-                <min>0.25</min>
-                <max>30.0</max>
-                <resolution>0.01</resolution>
-            </range>
-            <noise>
-                <type>gaussian</type>
-                <mean>0.0</mean>
-                <stddev>0.01</stddev>
-            </noise>
-        </ray>
-            <plugin name="gazebo_ros_head_hokuyo_controller" filename="libgazebo_ros_laser.so">
-                <topicName>/scan</topicName>
-                <frameName>lidar_link</frameName>
+    <xacro:macro name="bob_ros_gz">
+        <gazebo reference="base_link">
+            <material>Gazebo/Red</material>
+        </gazebo>
+        <gazebo reference="front_left_wheel">
+            <material>Gazebo/Black</material>
+        </gazebo>
+        <gazebo reference="front_right_wheel">
+            <material>Gazebo/Black</material>
+        </gazebo>
+        <gazebo reference="back_left_wheel">
+            <material>Gazebo/Black</material>
+        </gazebo>
+        <gazebo reference="back_right_wheel">
+            <material>Gazebo/Black</material>
+        </gazebo>
+        <gazebo reference="lidar_link">
+            <material>Gazebo/Black</material>
+        </gazebo>
+        <gazebo reference="camera_link">
+            <material>Gazebo/Black</material>
+        </gazebo>
+        <gazebo>
+            <plugin name="gz::sim::systems::DiffDrive" filename = "gz-sim-diff-drive-system">
+                <odom_publish_frequency>30</odom_publish_frequency>
+                <left_joint>front_left_wheel_joint</left_joint>
+                <left_joint>back_left_wheel_joint</left_joint>
+                <right_joint>front_right_wheel_joint</right_joint>
+                <right_joint>back_right_wheel_joint</right_joint>
+                <wheel_separation>0.35</wheel_separation>
+                <wheel_radius>0.1</wheel_radius>
+                <max_linear_acceleration>2</max_linear_acceleration>
+                <min_linear_acceleration>-2</min_linear_acceleration>
+                <max_angular_acceleration>3</max_angular_acceleration>
+                <min_angular_acceleration>-3</min_angular_acceleration>
+                <max_linear_velocity>0.5</max_linear_velocity>
+                <min_linear_velocity>-0.5</min_linear_velocity>
+                <max_angular_velocity>2.0</max_angular_velocity>
+                <min_angular_velocity>-2.0</min_angular_velocity>
+                <odom_topic>odom</odom_topic>
+                <frame_id>odom</frame_id>
+                <child_frame_id>base_footprint</child_frame_id>
+                <topic>cmd_vel</topic>
+                <tf_topic>tf</tf_topic>
             </plugin>
+        </gazebo>
+        <gazebo reference="lidar_link">
+            <sensor name="laser" type="gpu_lidar">
+                <visualize>false</visualize>
+                <update_rate>10</update_rate>
+                <lidar>
+                    <scan>
+                        <horizontal>
+                            <samples>360</samples>
+                            <min_angle>-3.14</min_angle>
+                            <max_angle>3.14</max_angle>
+                        </horizontal>
+                    </scan>
+                    <range>
+                        <min>0.3</min>
+                        <max>12</max>
+                    </range>
+                </lidar>
+                <topic>scan</topic>
+                <gz_frame_id>lidar_frame</gz_frame_id>
             </sensor>
-    </gazebo>
-    <gazebo reference="camera_link">
-        <sensor type="camera" name="camera">
-            <update_rate>30.0</update_rate>
-            <camera name="head">
-                <horizontal_fov>1.3962634</horizontal_fov>
-                <image>
-                    <width>800</width>
-                    <height>800</height>
-                    <format>R8G8B8</format>
-                </image>
+        </gazebo>
+        <gazebo reference="camera_link">
+            <sensor name="rgbd_camera" type="rgbd_camera">
+                <update_rate>15</update_rate>
+                <camera>
+                    <camera_info_topic>camera/camera_info</camera_info_topic>
+                    <horizontal_fov>1.05</horizontal_fov>
+                    <image>
+                        <width>640</width>
+                        <height>480</height>
+                        <format>R8G8B8</format>
+                    </image>
                     <clip>
-                    <near>0.02</near>
-                    <far>300</far>
-                </clip>
-                <noise>
-                    <type>gaussian</type>
-                    <mean>0.0</mean>
-                    <stddev>0.007</stddev>
-                </noise>
-            </camera>
-            <plugin name="camera_controller" filename="libgazebo_ros_camera.so">
-                <alwaysOn>true</alwaysOn>
-                <updateRate>0.0</updateRate>
-                <cameraName>/camera</cameraName>
-                <imageTopicName>image_raw</imageTopicName>
-                <cameraInfoTopicName>camera_info</cameraInfoTopicName>
-                <frameName>camera_optical_frame</frameName>
-                <hackBaseline>0.07</hackBaseline>
-                <distortionK1>0.0</distortionK1>
-                <distortionK2>0.0</distortionK2>
-                <distortionK3>0.0</distortionK3>
-                <distortionT1>0.0</distortionT1>
-                <distortionT2>0.0</distortionT2>
+                        <near>0.1</near>
+                        <far>8.0</far>
+                    </clip>
+                </camera>
+                <topic>camera</topic>
+                <gz_frame_id>kinect_depth_optical_frame</gz_frame_id>
+            </sensor>
+        </gazebo>
+        <gazebo>
+            <plugin name="joint_state_publisher" filename= "libgazebo_ros_joint_state_publisher.so">
+            <jointName>front_left_wheel_joint, front_right_wheel_joint, back_left_wheel_joint, back_right_wheel_joint</jointName>
             </plugin>
-        </sensor>
-    </gazebo>
-    <gazebo>
-        <plugin name="joint_state_publisher" filename= "libgazebo_ros_joint_state_publisher.so">
-        <jointName>front_left_wheel_joint, front_right_wheel_joint, back_left_wheel_joint, back_right_wheel_joint</jointName>
-        </plugin>
-    </gazebo>
+        </gazebo>
+    </xacro:macro>
 </robot>
