Commit message: attempt at fixing missing feedback

File: src/amr/lv1/robot_description/urdf/bob_ros_model_urdf.xacro (robot description, xacro)
@@ -73,5 +73,5 @@
             <parent link="base_link"/>
             <child link="lidar_link"/>
-            <origin rpy="0 0 3.14" xyz="0 0 .15"/>
+            <origin rpy="0 0 0" xyz="0 0 .15"/>
         </joint>
         <link name= "camera_link">
