Commit message: mock code

File: src/nrs/nrs_lv3_ws/src/ur5_robotiq_sim/urdf/ur5_robotiq_3f_gazebo.xacro (robot description, xacro)
@@ -18,4 +18,6 @@
     <xacro:include
         filename="$(find robotiq_description)/urdf/robotiq_3f_gripper_articulated_macro.xacro" />
+    <!-- Include FT300 macro -->
+    <xacro:include filename="$(find robotiq_description)/urdf/robotiq_ft300.urdf.xacro"/>
     <!-- Include UR macro -->
     <xacro:include filename="$(find ur_description)/urdf/ur_macro.xacro" />
@@ -36,4 +38,7 @@
         <origin xyz="0 0 0" rpy="0 0 0" />          <!-- position robot in the world -->
     </xacro:ur_robot>
+    <xacro:robotiq_ft300 parent="tool0" tf_prefix="$(arg tf_prefix)">
+        <origin xyz="0 0 -0.004" rpy="0 0 0"/>
+    </xacro:robotiq_ft300>
     <!-- Add gripper -->
     <xacro:robotiq_3f_gripper_articulated prefix="rq_" />
@@ -41,5 +46,5 @@
     <joint name="gripper_tool0_joint" type="fixed">
         <origin xyz="0 0 0.0535" rpy="${-pi/2} ${-pi} ${-pi/4}" />
-        <parent link="tool0" />
+        <parent link="robotiq_ft_frame_id" />
         <child link="rq_palm" />
     </joint>

File: src/nrs/nrs_lv3_ws/src/ur5_robotiq_sim/urdf/ur_gz.xacro (robot description, xacro)
@@ -6,4 +6,6 @@
         filename="$(find robotiq_description)/urdf/robotiq_3f_gripper_articulated_macro_fixed.xacro" />
     <xacro:include filename="$(find ur_simulation_gz)/urdf/ur_gz.ros2_control.xacro" />
+    <!-- Include FT300 macro -->
+    <xacro:include filename="$(find robotiq_description)/urdf/robotiq_ft300.urdf.xacro"/>
     <!-- possible 'ur_type' values: ur3, ur5, ur10, ur3e, ur5e, ur7e, ur10e, ur12e, ur16e, ur8long,
     ur15, ur20,
@@ -32,7 +34,7 @@
     <link name="table">
         <visual>
-            <origin xyz="0 0 0.4" rpy="0 0 0" />
+            <origin xyz="0 0 0.375" rpy="0 0 0" />
             <geometry>
-                <box size="1.0 2.0 0.8" />
+                <box size="0.8 1.8 0.75" />
             </geometry>
             <material name="brown">
@@ -41,11 +43,11 @@
         </visual>
         <collision>
-            <origin xyz="0 0 0.4" rpy="0 0 0" />
+            <origin xyz="0 0 0.375" rpy="0 0 0" />
             <geometry>
-                <box size="1.0 2.0 0.8" />
+                <box size="0.8 1.8 0.75" />
             </geometry>
         </collision>
         <inertial>
-            <origin xyz="0 0 0.4" rpy="0 0 0" />
+            <origin xyz="0 0 0.375" rpy="0 0 0" />
             <mass value="1.0" />
             <inertia
@@ -64,5 +66,5 @@
         <parent link="table" />
         <child link="robot_mount" />
-        <origin xyz="0 ${-(2.0/2 - 0.3)} 0.8" rpy="0 0 0" />
+        <origin xyz="0 ${-(1.8/2 - 0.445)} 0.75" rpy="0 0 ${pi}" />
     </joint>
     <!-- Wall to the right of the robot -->
@@ -71,5 +73,5 @@
             <origin xyz="0 0 1.0" rpy="0 0 0" />
             <geometry>
-                <box size="0.05 1.0 2.0" />
+                <box size="0.05 4.0 2.0" />
             </geometry>
             <material name="light_gray">
@@ -80,5 +82,5 @@
             <origin xyz="0 0 1.0" rpy="0 0 0" />
             <geometry>
-                <box size="0.05 1.0 2.0" />
+                <box size="0.05 4.0 2.0" />
             </geometry>
         </collision>
@@ -92,5 +94,5 @@
         <parent link="table" />
         <child link="wall" />
-        <origin xyz="${0.5+0.05/2} ${-(2.0/2 - 0.3)} 0.0" rpy="0 0 0" />
+        <origin xyz="${0.4+0.05/2} ${-(1.8/2 - 0.3)} 0.0" rpy="0 0 0" />
     </joint>
     <!-- arm -->
@@ -107,11 +109,22 @@
         <origin xyz="0 0 0" rpy="0 0 0" /> <!-- position robot in the robot_mount -->
     </xacro:ur_robot>
-    <!-- Robotiq gripper -->
+    <!-- Robotiq senzor -->
+    <xacro:robotiq_ft300 parent="tool0" tf_prefix="$(arg tf_prefix)">
+        <origin xyz="0 0 -0.004" rpy="0 0 0"/>
+    </xacro:robotiq_ft300>
+    <!-- Add gripper -->
     <xacro:robotiq_3f_gripper_articulated prefix="$(arg rq_prefix)" />
-    <!-- Attach gripper to tool0 -->
+    <!-- Attach gripper to UR5 tool0 -->
     <joint name="tool0_$(arg rq_prefix)palm_joint" type="fixed">
-        <parent link="tool0" />
+        <origin xyz="0 0 0.0535" rpy="${-pi/2} ${-pi} ${-pi/4}" />
+        <parent link="robotiq_ft_frame_id" />
         <child link="$(arg rq_prefix)palm" />
-        <origin xyz="0 0 0.0535" rpy="${-pi/2} ${-pi} ${-pi/4}" />
+    </joint>
+    <link name="gripper"/>
+    <!-- Gripper tf to UR5 tool0 -->
+    <joint name="$(arg rq_prefix)palm_joint_gripper" type="fixed">
+        <origin xyz="-0.075 0.13 0" rpy="0 0 0" />
+        <parent link="$(arg rq_prefix)palm" />
+        <child link="gripper" />
     </joint>
     <gazebo reference="robot_mount"> </gazebo>
